File: STM32.kicad_pcb (KiCad board)
At the start: 4 copper layers, 44 parts, among them J1 USB_C_Receptacle_USB2.0_16P, J2 Conn_ARM_SWD_TagConnect_TC2030, J3 Conn_Coaxial, J4 Conn_01x04_Pin, SW1 SW_Push, U1 AMS1117-3.3, U2 STM32WB55CEUx, Y1 Crystal_32.768kHz, Y2 Crystal_32MHz

Commit message: design-compleat; verificaton,revision-remaning
Parts:
- R6, R7, Y1: moved to B.Cu
- moved C3 84.5 mm to (67.3, 101.9), turned to -90 degrees
- moved C17 77.1 mm to (73.0, 96.5), turned to 180 degrees
- moved C19 76.4 mm to (73.2, 106.3), turned to -90 degrees
- moved C18 73.9 mm to (76.5, 96.5)
- moved J4 73.2 mm to (73.6, 78.9), turned to 180 degrees
- moved C4 72.2 mm to (69.0, 101.6), turned to -90 degrees
- moved C6 71.9 mm to (71.9, 101.6), turned to -90 degrees
- moved C5 71.0 mm to (70.4, 101.6), turned to -90 degrees
- moved C7 70.5 mm to (73.4, 101.6), turned to -90 degrees
- moved C13 70.4 mm to (76.5, 101.6), turned to -90 degrees
- moved D3 70.1 mm to (81.9, 108.8), turned to 90 degrees
- moved C8 69.2 mm to (74.8, 101.6), turned to -90 degrees
- moved C10 68.2 mm to (86.0, 94.2), turned to 90 degrees
- moved U1 66.0 mm to (73.9, 86.5), turned to 180 degrees
- moved C16 64.9 mm to (84.9, 109.7), turned to 180 degrees
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Routing:
- net P,+3.3: track 0.00 -> 147.1 mm, vias 0 -> 15
- net GND: track 0.00 -> 56.7 mm, vias 0 -> 128
- net Net-(C13-+): track 0.00 -> 53.3 mm, vias 0 -> 2
- net P,+5: track 0.00 -> 46.2 mm, vias 0 -> 3
- net Net-(J4-Pin_3): track 0.00 -> 40.0 mm
- net Net-(J4-Pin_2): track 0.00 -> 32.6 mm
- net Net-(D2-L1-Pad1): track 0.00 -> 25.1 mm
- net Net-(D2-L2-Pad3): track 0.00 -> 20.6 mm
- net Net-(R10-Pad2): track 0.00 -> 20.3 mm
- net Net-(J2-SWO): track 0.00 -> 16.4 mm
- net Net-(J2-SWCLK): track 0.00 -> 14.5 mm
- net /BOOT0: track 0.00 -> 13.8 mm, vias 0 -> 2
- net Net-(C1-+): track 0.00 -> 12.7 mm
- net Net-(U2-OSC_OUT): track 0.00 -> 9.48 mm
- net Net-(J2-SWDIO): track 0.00 -> 8.41 mm
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- added copper zone on In1.Cu, net GND
- added copper zone on In2.Cu, net GND
Other:
- board outline added: 31.4 x 50.1 mm

Commit message: revision-1
Routing:
- net P,+3.3: track 147.1 -> 149.3 mm
Changed lines of the file:
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@@
+	)
+	(segment
+		(start 87.84 98.11)
+		(end 88.82 98.11)
+		(width 0.19)
+		(layer "B.Cu")
+		(net 3)
 	)
 	(segment
@@
 		(layer "B.Cu")
 		(net 3)
+	)
+	(segment
+		(start 88.82 98.11)
+		(end 89.69 97.24)
+		(width 0.19)
+		(layer "B.Cu")
+		(net 3)

Commit message: added test points
Parts:
- added FID1: Fiducial_0.5mm, PCM_SparkFun-Aesthetic:Fiducial_0.5mm_Mask1mm, F.Cu at (66.3, 107.4)
- added FID2: Fiducial_0.5mm, PCM_SparkFun-Aesthetic:Fiducial_0.5mm_Mask1mm, F.Cu at (95.1, 76.1)
- added FID3: Fiducial_0.5mm, PCM_SparkFun-Aesthetic:Fiducial_0.5mm_Mask1mm, F.Cu at (90.2, 118.5)
- added H1: MountingHole_Pad, MountingHole:MountingHole_2.2mm_M2_DIN965_Pad, F.Cu at (93.6, 72.7)
- added H2: MountingHole_Pad, MountingHole:MountingHole_2.2mm_M2_DIN965_Pad, F.Cu at (93.4, 116.7)
- added H4: MountingHole_Pad, MountingHole:MountingHole_2.2mm_M2_DIN965_Pad, F.Cu at (67.7, 80.8)
- added TP1: TestPoint, TestPoint:TestPoint_Pad_D1.0mm, F.Cu at (80.4, 88.4)
- added TP10: TestPoint, TestPoint:TestPoint_Pad_D1.0mm, F.Cu at (94.8, 102.1)
- added TP13: TestPoint, TestPoint:TestPoint_Pad_D1.0mm, F.Cu at (78.2, 99.9)
- added TP14: TestPoint, TestPoint:TestPoint_Pad_D1.0mm, B.Cu at (88.6, 95.4)
- added TP15: TestPoint, TestPoint:TestPoint_Pad_D1.0mm, B.Cu at (88.9, 93.0)
- added TP16: TestPoint, TestPoint:TestPoint_Pad_D1.0mm, F.Cu at (94.8, 88.4)
- added TP17: TestPoint, TestPoint:TestPoint_Pad_D1.0mm, F.Cu at (93.0, 90.3)
- added TP19: TestPoint, TestPoint:TestPoint_Pad_D1.0mm, B.Cu at (86.1, 92.0)
- added TP2: TestPoint, TestPoint:TestPoint_Pad_D1.0mm, F.Cu at (83.2, 93.2)
- added TP21: TestPoint, TestPoint:TestPoint_Pad_D1.0mm, B.Cu at (77.1, 90.7)
- added TP22: TestPoint, TestPoint:TestPoint_Pad_D1.0mm, B.Cu at (88.3, 99.5)
- added TP3: TestPoint, TestPoint:TestPoint_Pad_D1.0mm, B.Cu at (84.4, 92.2)
- added TP4: TestPoint, TestPoint:TestPoint_Pad_D1.0mm, F.Cu at (90.8, 88.9)
- added TP6: TestPoint, TestPoint:TestPoint_Pad_D1.0mm, B.Cu at (91.7, 86.0)
- added TP7: TestPoint, TestPoint:TestPoint_Pad_D1.0mm, F.Cu at (94.8, 97.4)
- added TP8: TestPoint, TestPoint:TestPoint_Pad_D1.0mm, B.Cu at (85.3, 106.0)
- added TP9: TestPoint, TestPoint:TestPoint_Pad_D1.0mm, F.Cu at (83.3, 111.1)
- C19: value 19 -> 100n
- moved J4 2.11 mm to (75.1, 77.4)
Routing:
- net /SMPS_FB: track 6.75 -> 9.44 mm
- net Net-(J4-Pin_3): track 40.0 -> 42.1 mm
- net Net-(J4-Pin_2): track 32.6 -> 34.6 mm
- net /RF: track 2.90 -> 4.90 mm
- net P,+3.3: track 149.3 -> 151.1 mm, vias 15 -> 16
- net GND: track 56.7 -> 58.4 mm, vias 128 -> 125
- net Net-(C15-+): track 4.18 -> 5.32 mm, vias 0 -> 1
- net Net-(J2-SWDIO): track 8.41 -> 9.23 mm, vias 0 -> 1
- net /USB_D+: track 7.58 -> 8.27 mm, vias 0 -> 1
- net Net-(C1-+): vias 0 -> 1
- net /USB_D-: vias 0 -> 1
- net /SMPSLX: vias 0 -> 1

Commit message: revision-2
Parts:
- TP2: moved to B.Cu
- moved TP13 6.08 mm to (74.0, 104.3)
- moved TP3 2.03 mm to (84.4, 94.3)
- moved TP21 1.80 mm to (78.9, 90.7)
- moved TP6 1.77 mm to (93.0, 84.8)
- moved TP14 1.71 mm to (90.2, 95.7)
- moved TP4 1.44 mm to (91.1, 87.5)
- moved TP2 1.13 mm to (82.3, 93.9), turned to 180 degrees
- moved TP19 0.97 mm to (86.1, 93.0)
- moved TP1 0.12 mm to (80.2, 88.4)
Routing:
- net GND: track 58.4 -> 48.7 mm, vias 125 -> 102
- net Net-(C13-+): track 53.3 -> 55.7 mm
- net P,+5: track 46.2 -> 48.4 mm
- net /BOOT0: track 13.8 -> 15.9 mm
- net Net-(J2-SWDIO): track 9.23 -> 11.3 mm
- net Net-(C1-+): track 12.7 -> 14.5 mm
- net /USB_D-: track 6.08 -> 7.88 mm
- net Net-(J2-SWCLK): track 14.5 -> 15.8 mm, vias 0 -> 1
- net P,+3.3: track 151.1 -> 152.1 mm
- net Net-(U2-PA2): track 7.76 -> 8.65 mm
Other:
- rule pad_to_mask_clearance: 0.8 -> 0
