File: STM32.kicad_sch (KiCad schematic)
At the start: 44 parts, among them J1 USB_C_Receptacle_USB2.0_16P, J2 Conn_ARM_SWD_TagConnect_TC2030, J3 Conn_Coaxial, J4 Conn_01x04_Pin, SW1 SW_Push, U1 AMS1117-3.3, U2 STM32WB55CEUx, Y1 Crystal_32.768kHz, Y2 Crystal_32MHz

Commit message: design-compleat; verificaton,revision-remaning
Parts:
- C19: value 19 -> 100n
Changed lines of the file:
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@@
 			)
 		)
-		(property "Value" "19"
+		(property "Value" "100n"
 			(at 233.68 133.3499 0)
 			(effects

Commit message: added test points
Parts:
- added FID1, FID2, FID3: Fiducial_0.5mm, PCM_SparkFun-Aesthetic:Fiducial_0.5mm_Mask1mm, symbol PCM_SparkFun-Aesthetic:Fiducial_0.5mm
- added H1, H2, H3, H4: MountingHole_Pad, MountingHole:MountingHole_2.2mm_M2_DIN965_Pad, symbol Mechanical:MountingHole_Pad
- added TP1, TP10, TP11, TP12, TP13, TP14, TP15, TP16, TP17, TP18, TP19, TP2, TP21, TP22, TP23, TP3, TP4, TP5, TP6, TP7, TP8, TP9: TestPoint, TestPoint:TestPoint_Pad_D1.0mm, symbol Connector:TestPoint
Connections:
- net BOOT0: now also TP13.1, TP23.1
- net GND: now also H1.1, H2.1, H3.1, H4.1, TP7.1
- net P,+3.3: now also TP18.1, TP19.1, TP5.1
- net P,+5: now also TP6.1
- net RF: now also TP9.1
- net SMPSLX: now also TP22.1
- net SMPS_FB: now also TP10.1
- net USB_D+: now also TP15.1
- net USB_D-: now also TP14.1
- net at C18.1 (+), U2.2 (PC14), Y1.2: now also TP11.1
- net at C15.1 (+), L3.1 (+), U2.21 (RF1): now also TP8.1
- net at C17.1 (+), U2.3 (PC15), Y1.1: now also TP12.1
- net at J2.2 (SWDIO), U2.39 (PA13): now also TP3.1
- net at J2.4 (SWCLK), U2.41 (PA14): now also TP2.1
- net at J2.6 (SWO), U2.43 (PB3): now also TP1.1
- net at C13.1 (+), J2.3 (~{RESET}), U2.7 (NRST): now also TP4.1
- net at C1.1 (+), R1.2, R2.2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: now also TP21.1
- net at D2.1 (L1), J1.A7 (D-), J1.B7 (D-): now also TP16.1
- net at D2.3 (L2), J1.A6 (D+), J1.B6 (D+): now also TP17.1

Commit message: revision-2
Parts:
- removed H3: MountingHole_Pad, MountingHole:MountingHole_2.2mm_M2_DIN965_Pad, symbol Mechanical:MountingHole_Pad
- removed TP11, TP12, TP18, TP23, TP5: TestPoint, TestPoint:TestPoint_Pad_D1.0mm, symbol Connector:TestPoint
